Commit message: updated launch files with realsense, moveit, camera static tf, pointcloud in rviz. removing octree from point cloud planning scene for now. updated urdf in .xacro file to align world and yumi_body

File: catkin_ws/src/config/descriptions/urdf/yumi_setup.urdf.xacro (robot description, xacro)
@@ -14,6 +14,9 @@
   <link name="world"/>
   <!--yumi-->
+<!--   <xacro:yumi name="yumi" hardware_interface="$(arg prefix)" parent="world" limits="experimental">
+    <origin xyz="0 0 0.1" rpy="0 0 0" />
+  </xacro:yumi> -->
   <xacro:yumi name="yumi" hardware_interface="$(arg prefix)" parent="world" limits="experimental">
-    <origin xyz="0 0 0.1" rpy="0 0 0" />
+    <origin xyz="0 0 0" rpy="0 0 0" />
   </xacro:yumi>
   <xacro:property name="gripper" value="$(arg gripper)" />
